File: circadian rev2.0/circadian rev2.0.brd (EAGLE design)
At the start: 174 x 111.4 mm, 244 parts, among them IC1 4017D, IC10 LM4040B05, IC2 4051D, IC3 4051D, IC4 74HC595D, IC5 4053D, IC6 74HC595D, IC7 4051D, IC8 FT232RL, IC9 LM4040B10

Commit message: Add files via upload
Connections:
- removed net N$80: C21.2, LED65.1, LED66.3
- new net N$116: LED65.1, LED66.3
- net LED_POWER: now also C13.1, C14.1, C15.1, C16.1, C17.1, C18.1, C19.1, C20.1, C21.2, C22.2
- net N$12: no longer C14.1
- net N$13: no longer C15.1
- net N$22: no longer C13.1
- net N$38: no longer C16.1
- net N$39: no longer C17.1
- net N$57: no longer C18.1
- net N$58: no longer C20.1
- net N$76: no longer C19.1
- net N$86: no longer C22.2
Routing:
- net LED_POWER: track 988.7 -> 1058.3 mm
- net N$116: track 0.00 -> 25.9 mm
- net N$80: track 25.7 -> 0.00 mm
- net N$22: track 22.1 -> 11.2 mm
- net N$39: track 19.9 -> 11.5 mm
- net N$13: track 19.9 -> 11.5 mm
- net N$58: track 19.3 -> 12.2 mm
- net N$38: track 18.3 -> 14.9 mm
- net N$76: track 18.4 -> 15.0 mm
- net N$86: track 16.2 -> 19.5 mm
- net N$57: track 18.4 -> 15.0 mm
- net N$12: track 18.3 -> 15.2 mm
