File: circadian rev2.1/circadian rev2.1.brd (EAGLE design)
At the start: 174 x 111.4 mm, 246 parts, among them IC1 4017D, IC10 LM4040B05, IC2 4051D, IC3 4051D, IC4 74HC595D, IC5 4053D, IC6 74HC595D, IC7 4051D, IC8 FT232RL, IC9 LM4040B10

Commit message: Fixed wrong LED type causing confusion
Parts:
- LED1, LED10, LED11, LED12, LED13, LED14, LED15, LED16, LED17, LED18, LED19, LED2, LED20, LED21, LED22, LED23, LED24, LED25, LED26, LED27, LED28, LED29, LED3, LED30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: value WS2812B3535 -> SK68123535
